File: pcb/skibidi-digital-vinyl.kicad_sch (KiCad schematic)
At the start: 0 parts

Commit message: finished disc schematic, might add testpoints later to make full use of the ch32v003
Parts:
- added C1, C2: 0.1u, Capacitor_SMD:C_0402_1005Metric, symbol Device:C
- added C3: 1u, Capacitor_SMD:C_0402_1005Metric, symbol Device:C
- added R1: 10k, Resistor_SMD:R_0603_1608Metric, symbol Device:R
- added U1: CH32V003FxUx, Package_DFN_QFN:QFN-20-1EP_3x3mm_P0.4mm_EP1.65x1.65mm, symbol MCU_WCH_RiscV:CH32V003FxUx
- added U2: BY25Q32ESHIG(R), easyeda2kicad:DFN-8_L4.0-W3.0-P0.80-TL-EP_GT5YL24A1Y520, symbol easyeda2kicad:BY25Q32ESHIG(R)
Connections:
- new net +3V3: C1.1, C2.1, C3.1, R1.1, U1.6 (VDD), U2.3 (~{WP}(IO2)), U2.7 (~{HOLD}/(IO3)), U2.8 (VCC)
- new net CS: U1.8 (PC1), U2.1 (~{CS})
- new net GND: C1.2, C2.2, C3.2, U1.21 (VSS), U1.4 (VSS), U2.10 (EP), U2.4 (VSS), U2.9 (EP)
- new net LED: U1.18 (PD4)
- new net MISO: U1.14 (PC7), U2.2 (SO(IO1))
- new net MOSI: U1.13 (PC6), U2.5 (SI(IO0))
- new net RESET: R1.2, U1.1 (PD7)
- new net SCK: U1.12 (PC5), U2.6 (SCLK)
- new net SWIO: U1.15 (PD1)
- new net UART_RX: U1.20 (PD6)
- new net UART_TX: U1.19 (PD5)

Commit message: disc routing done
Parts:
- added D1: LED, LED_SMD:LED_0603_1608Metric, symbol Device:LED
- added R2: 1k, Resistor_SMD:R_0603_1608Metric, symbol Device:R
- added TP1, TP2, TP3, TP4, TP5: TestPoint, TestPoint:TestPoint_Pad_D1.0mm, symbol Connector:TestPoint
Connections:
- net +3V3: now also R1.2; no longer R1.1
- net GND: now also D1.1 (K)
- net LED: now also R2.1
- net RESET: now also R1.1; no longer R1.2
- net SWIO: now also TP1.1
- net at U1.11 (PC4): now also TP4.1
- net at U1.16 (PD2): now also TP2.1
- net at U1.17 (PD3): now also TP3.1
- net at U1.2 (PA1): now also TP5.1
- new net: D1.2 (A), R2.2
Other:
- moved on the sheet: R1

Commit message: update silkscreen text
Other:
- company: (none) -> Toby Cm's Lab x Hack Club
- title: (none) -> Skibidi Digital Vinyl Disc
Changed lines of the file:
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@@
 	(generator_version "9.0")
 	(paper "A4")
+	(title_block
+		(title "Skibidi Digital Vinyl Disc")
+		(date "2026-01-31")
+		(rev "A")
+		(company "Toby Cm's Lab x Hack Club")
+	)
 	(junction
 		(at 88.9 124.46)
