File: disc_pcb/skibidi-digital-vinyl-disc.kicad_pcb (KiCad board)
At the start: 2 copper layers, 100 x 100 mm, 13 parts, among them U1 CH32V003FxUx, U2 BY25Q32ESHIG(R)

Commit message: update
Parts:
- turned R1 to 90 degrees
Routing:
- net /UART_RX: track 25.9 -> 14.4 mm
- net /UART_TX: track 20.2 -> 11.0 mm
- net GND: track 8.00 -> 0.00 mm
- net Net-(D1-A): track 0.00 -> 2.04 mm
