File: player_pcb/skibidi-digital-vinyl-player.kicad_sch (KiCad schematic)
At the start: 28 parts, among them SW1 TS-1088-AR02016, SW2 TS-1088-AR02016, U1 RP2040, U4 BY25Q32ESHIG(R), U5 ABM8-272-T3, U6 ME6211C33M5

Commit message: second to done
Parts:
- added LS1, LS2: Speaker, symbol Device:Speaker
- added SW3, SW4, SW5, SW6, SW7: SW_Push, PCM_marbastlib-mx:SW_MX_1u, symbol Switch:SW_Push
Connections:
- net GND: now also SW3.2, SW4.2, SW5.2, SW6.2, SW7.2
- net at U1.11 (GPIO8): now also SW4.1
- net at U1.12 (GPIO9): now also SW5.1
- net at U1.13 (GPIO10): now also SW6.1
- net at U1.14 (GPIO11): now also SW7.1
- net DAC/DIN: now reaches U1.4 (GPIO2)
- net DAC/BCK: now reaches U1.5 (GPIO3)
- net DAC/WS: now reaches U1.6 (GPIO4)
- net Amplifier/~{RUN}: now reaches U1.7 (GPIO5)
- net at U1.9 (GPIO7): now also SW3.1
- new net Amplifier/LOUT+: LS1.1
- new net Amplifier/LOUT-: LS1.2
- new net Amplifier/ROUT+: LS2.1
- new net Amplifier/ROUT-: LS2.2
Other:
- added sheet USB (usb.kicad_sch)
- sheet Amplifier ports: added INL, INR, LOUT+, LOUT-, ROUT+, ROUT-, ~{RUN}; removed none
- sheet DAC ports: added BCK, DIN, LCH, RCH, WS; removed none

Commit message: update
Parts:
- added C32: 100n, Capacitor_SMD:C_0402_1005Metric, symbol Device:C
- added J1: Conn_02x04_Odd_Even, Connector_JST:JST_XH_S8B-XH-A_1x08_P2.50mm_Horizontal, symbol Connector_Generic:Conn_02x04_Odd_Even
- added R10: 330, Resistor_SMD:R_0603_1608Metric, symbol Device:R
- added R11, R12: 10k, Resistor_SMD:R_0603_1608Metric, symbol Device:R
- added TP1, TP2, TP3, TP4, TP8: TestPoint, TestPoint:TestPoint_Pad_D1.0mm, symbol Connector:TestPoint
- C22, C23: footprint (none) -> Capacitor_SMD:C_0402_1005Metric; LCSC Part # (none) -> C1549
- LS1, LS2: footprint (none) -> Connector_PinSocket_2.54mm:PinSocket_1x02_P2.54mm_Vertical
Connections:
- net +3V3: now also J1.2 (Pin_2), R12.2, TP8.1
- net GND: now also SW1.1, SW2.1, C32.2, J1.1 (Pin_1), J1.3 (Pin_3), J1.5 (Pin_5), J1.7 (Pin_7), J1.8 (Pin_8), R11.1; no longer R6.1, R7.1
- net QSPI_SS: now also R7.2; no longer SW2.2
- net RUN: now also R6.2, C32.1, R12.1; no longer SW1.2
- net at U1.15 (GPIO12): now also R10.1, R11.2
- net UART_TX: now reaches U1.2 (GPIO0)
- net UART_TX: now also J1.4 (Pin_4)
- net UART_RX: now reaches U1.3 (GPIO1)
- net UART_RX: now also J1.6 (Pin_6)
- net at U1.38 (GPIO26/ADC0): now also TP1.1
- net at U1.39 (GPIO27/ADC1): now also TP2.1
- net at U1.40 (GPIO28/ADC2): now also TP3.1
- net at U1.41 (GPIO29/ADC3): now also TP4.1
- net USB_D+ renamed USB/D-
- net USB_D- renamed USB/D+
- new net: R7.1, SW2.2
- new net: R6.1, SW1.2
- new net Neopixel/DIN: R10.2
Other:
- added sheet Neopixel (neopixel.kicad_sch)
- sheet USB ports: added D+, D-; removed none
- note added: "Daughter board"
- note added: "Decoupling capacitors"
- note added: "RUN filter"
- note added: "ring 1 (inner): 3.3V ring 2: UART TX on disc ring 3: UART RX on disc ring 4 (outer): GND daughter board holds pogo pins"
- moved on the sheet: R6, R7, SW1, SW2
