File: player_pcb/usb.kicad_sch (KiCad schematic)
At the start: 0 parts

Commit message: update
Parts:
- added D1: SS54, Diode_SMD:D_SMA, symbol Device:D_Schottky
- added D2: 5V, Diode_SMD:D_SOD-523, symbol Device:D_TVS
- added F1: 2A, Fuse:Fuse_1206_3216Metric, symbol Device:Polyfuse
- added FB1: 220Ω@100MHz, Resistor_SMD:R_0805_2012Metric_Pad1.20x1.40mm_HandSolder, symbol Device:FerriteBead
- added R8, R9: 5.1k, Resistor_SMD:R_0603_1608Metric, symbol Device:R
- added TP5, TP6, TP7: TestPoint, TestPoint:TestPoint_Pad_D1.0mm, symbol Connector:TestPoint
- added USB1: TYPE-C 16PIN 2MD(073), easyeda2kicad:USB-C-SMD_TYPE-C-6PIN-2MD-073, symbol easyeda2kicad:TYPE-C16PIN2MD(073)
Connections:
- new net: F1.1, USB1.11 (VBUS), USB1.2 (VBUS)
- new net: D1.2 (A), D2.1 (A1), F1.2
- new net: D1.1 (K), FB1.1, TP5.1
- new net: R9.2, USB1.10 (CC2)
- new net: R8.2, USB1.4 (CC1)
- new net D+: USB1.6 (DP1), USB1.8 (DP2)
- new net D-: USB1.5 (DN2), USB1.7 (DN1)
- new net GND: D2.2 (A2), R8.1, R9.1, TP7.1, USB1.1 (GND), USB1.12 (GND), USB1.13 (SHELL), USB1.14 (SHELL)
- new net VBUS: FB1.2, TP6.1
